File: HM2.kicad_pcb (KiCad board)
At the start: 2 copper layers, 85 parts, among them J1 Conn_01x05_Male, Q1 2SK880, Q2 2SC2713, Q3 2SA1163, Q4 2SC2713, U1 TL072, U2 TL072, U3 TL072

Commit message: PCB send to prod
Routing:
- net GND: vias 16 -> 49
Other:
- board outline added: 39.1 x 57 mm
- board text added: "9V"
- board text added: "DIST"
- board text added: "GND"
- board text added: "HIGH"
- board text added: "HM2 Clone V2"
- board text added: "IN"
- board text added: "LED"
- board text added: "LOW"
- board text added: "MID"
- board text added: "OUT"
- board text added: "VOL"
Changed lines of the file:
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@@
     (property "Sheetname" "")
     (attr through_hole)
-    (fp_text reference "RV4" (at 2.3 2.325 90 unlocked) (layer "F.SilkS")
+    (fp_text reference "RV4" (at 2.1 5.425 90 unlocked) (layer "F.SilkS")
       (effects (font (size 0.8128 0.8128) (thickness 0.1524)))
     )
@@
     (property "Sheetname" "")
     (attr through_hole)
-    (fp_text reference "RV1" (at 2.6 2.44 90 unlocked) (layer "F.SilkS")
+    (fp_text reference "RV1" (at 2.4 5.44 90 unlocked) (layer "F.SilkS")
       (effects (font (size 0.8128 0.8128) (thickness 0.1524)))
     )
@@
     (property "Sheetname" "")
     (attr through_hole)
-    (fp_text reference "RV3" (at 2.4 1.225 90 unlocked) (layer "F.SilkS")
+    (fp_text reference "RV3" (at 2.4 5.425 90 unlocked) (layer "F.SilkS")
       (effects (font (size 0.8128 0.8128) (thickness 0.1524)))
     )
@@
       (rotate (xyz 0 0 0))
     )
+  )
+  (gr_line (start 114.26066 147.1) (end 114.3 93.4) (layer "Edge.Cuts") (width 0.0381))
+  (gr_arc (start 114.3 93.1) (mid 114.73934 92.03934) (end 115.8 91.6) (layer "Edge.Cuts") (width 0.0381))
+  (gr_line (start 153.4 147.4) (end 153.4 93) (layer "Edge.Cuts") (width 0.0381))
+  (gr_arc (start 115.76066 148.6) (mid 114.7 148.16066) (end 114.26066 147.1) (layer "Edge.Cuts") (width 0.0381))
+  (gr_line (start 115.8 91.6) (end 151.9 91.6) (layer "Edge.Cuts") (width 0.0381))
+  (gr_line (start 115.76066 148.6) (end 152.3 148.6) (layer "Edge.Cuts") (width 0.0381))
+  (gr_arc (start 151.9 91.6) (mid 152.948087 91.98062) (end 153.4 93) (layer "Edge.Cuts") (width 0.0381))
+  (gr_arc (start 153.4 147.4) (mid 153.131162 148.257732) (end 152.3 148.6) (layer "Edge.Cuts") (width 0.0381))
+  (gr_line (start 114.3 93.4) (end 114.3 93.1) (layer "Edge.Cuts") (width 0.0381))
+  (gr_text "HM2 Clone\nV2" (at 134 104.3) (layer "F.SilkS")
+    (effects (font (size 0.8128 0.8128) (thickness 0.1524)))
+  )
+  (gr_text "9V" (at 127.5 148.5) (layer "F.SilkS")
+    (effects (font (size 0.8128 0.8128) (thickness 0.1524)))
+  )
+  (gr_text "MID" (at 133.9 92.4) (layer "F.SilkS")
+    (effects (font (size 0.8128 0.8128) (thickness 0.1524)))
+  )
+  (gr_text "HIGH" (at 148.9 107.9 90) (layer "F.SilkS")
+    (effects (font (size 0.8128 0.8128) (thickness 0.1524)))
+  )
+  (gr_text "GND" (at 137.6 148.7) (layer "F.SilkS")
+    (effects (font (size 0.8128 0.8128) (thickness 0.1524)))
+  )
+  (gr_text "DIST" (at 119.3 106.5 90) (layer "F.SilkS")
+    (effects (font (size 0.8128 0.8128) (thickness 0.1524)))
+  )
+  (gr_text "VOL" (at 148.3 133.9 90) (layer "F.SilkS")
+    (effects (font (size 0.8128 0.8128) (thickness 0.1524)))
+  )
+  (gr_text "OUT\n" (at 135.1 148.7) (layer "F.SilkS")
+    (effects (font (size 0.8128 0.8128) (thickness 0.1524)))
+  )
+  (gr_text "LED" (at 132.5 148.7) (layer "F.SilkS")
+    (effects (font (size 0.8128 0.8128) (thickness 0.1524)))
+  )
+  (gr_text "IN" (at 130 148.6) (layer "F.SilkS")
+    (effects (font (size 0.8128 0.8128) (thickness 0.1524)))
+  )
+  (gr_text "LOW" (at 119.2 97.6 90) (layer "F.SilkS")
+    (effects (font (size 0.8128 0.8128) (thickness 0.1524)))
   )
   (segment (start 138.8 143.2) (end 136.9 141.3) (width 0.3) (layer "F.Cu") (net 1))
@@
   (segment (start 133.9 120.6) (end 137.3 124) (width 0.6) (layer "B.Cu") (net 6))
   (segment (start 136.2 107.5) (end 136.2 98.2) (width 0.6) (layer "B.Cu") (net 6))
+  (via (at 120.4 102) (size 0.6) (drill 0.3) (layers "F.Cu" "B.Cu") (free) (net 7))
+  (via (at 151 100.9) (size 0.6) (drill 0.3) (layers "F.Cu" "B.Cu") (free) (net 7))
+  (via (at 151.2 138.9) (size 0.6) (drill 0.3) (layers "F.Cu" "B.Cu") (free) (net 7))
+  (via (at 116.1 140.7) (size 0.6) (drill 0.3) (layers "F.Cu" "B.Cu") (free) (net 7))
+  (via (at 137 143.4) (size 0.6) (drill 0.3) (layers "F.Cu" "B.Cu") (free) (net 7))
+  (via (at 116.9 102) (size 0.6) (drill 0.3) (layers "F.Cu" "B.Cu") (free) (net 7))
+  (via (at 122.8 102) (size 0.6) (drill 0.3) (layers "F.Cu" "B.Cu") (free) (net 7))
+  (via (at 144.7 132.5) (size 0.6) (drill 0.3) (layers "F.Cu" "B.Cu") (free) (net 7))
+  (via (at 116.1 145.5) (size 0.6) (drill 0.3) (layers "F.Cu" "B.Cu") (free) (net 7))
   (via (at 147.7 119.5) (size 0.6) (drill 0.3) (layers "F.Cu" "B.Cu") (free) (net 7))
+  (via (at 144.7 137.4) (size 0.6) (drill 0.3) (layers "F.Cu" "B.Cu") (free) (net 7))
+  (via (at 120.4 99.2) (size 0.6) (drill 0.3) (layers "F.Cu" "B.Cu") (free) (net 7))
+  (via (at 116.5 122.9) (size 0.6) (drill 0.3) (layers "F.Cu" "B.Cu") (free) (net 7))
   (via (at 129.8 111.6) (size 0.6) (drill 0.3) (layers "F.Cu" "B.Cu") (free) (net 7))
-  (via (at 143.6 132.7) (size 0.6) (drill 0.3) (layers "F.Cu" "B.Cu") (free) (net 7))
+  (via (at 143.4 132.5) (size 0.6) (drill 0.3) (layers "F.Cu" "B.Cu") (free) (net 7))
+  (via (at 116.5 132.1) (size 0.6) (drill 0.3) (layers "F.Cu" "B.Cu") (free) (net 7))
+  (via (at 122.8 107.8) (size 0.6) (drill 0.3) (layers "F.Cu" "B.Cu") (free) (net 7))
   (via (at 136.5 115.8) (size 0.6) (drill 0.3) (layers "F.Cu" "B.Cu") (free) (net 7))
+  (via (at 147.3 139.8) (size 0.6) (drill 0.3) (layers "F.Cu" "B.Cu") (free) (net 7))
+  (via (at 120.4 107.8) (size 0.6) (drill 0.3) (layers "F.Cu" "B.Cu") (free) (net 7))
+  (via (at 122.8 110.2) (size 0.6) (drill 0.3) (layers "F.Cu" "B.Cu") (free) (net 7))
+  (via (at 116.5 119.3) (size 0.6) (drill 0.3) (layers "F.Cu" "B.Cu") (free) (net 7))
   (via (at 131 136.6) (size 0.6) (drill 0.3) (layers "F.Cu" "B.Cu") (free) (net 7))
   (via (at 143.9 138.7) (size 0.6) (drill 0.3) (layers "F.Cu" "B.Cu") (free) (net 7))
+  (via (at 151 109.5) (size 0.6) (drill 0.3) (layers "F.Cu" "B.Cu") (free) (net 7))
   (via (at 116.5 129.9) (size 0.6) (drill 0.3) (layers "F.Cu" "B.Cu") (free) (net 7))
+  (via (at 140.1 93.1) (size 0.6) (drill 0.3) (layers "F.Cu" "B.Cu") (free) (net 7))
   (via (at 116.5 127.2) (size 0.6) (drill 0.3) (layers "F.Cu" "B.Cu") (free) (net 7))
+  (via (at 119.3 135.8) (size 0.6) (drill 0.3) (layers "F.Cu" "B.Cu") (free) (net 7))
   (via (at 134.9 116.7) (size 0.6) (drill 0.3) (layers "F.Cu" "B.Cu") (free) (net 7))
+  (via (at 147.2 135) (size 0.6) (drill 0.3) (layers "F.Cu" "B.Cu") (free) (net 7))
+  (via (at 151 93.1) (size 0.6) (drill 0.3) (layers "F.Cu" "B.Cu") (free) (net 7))
+  (via (at 147.2 132.4) (size 0.6) (drill 0.3) (layers "F.Cu" "B.Cu") (free) (net 7))
+  (via (at 119.3 128.5) (size 0.6) (drill 0.3) (layers "F.Cu" "B.Cu") (free) (net 7))
   (via (at 116.4 137.3) (size 0.6) (drill 0.3) (layers "F.Cu" "B.Cu") (free) (net 7))
   (via (at 143.2 125.9) (size 0.6) (drill 0.3) (layers "F.Cu" "B.Cu") (free) (net 7))
   (via (at 129.7 102) (size 0.6) (drill 0.3) (layers "F.Cu" "B.Cu") (free) (net 7))
+  (via (at 120.4 110.2) (size 0.6) (drill 0.3) (layers "F.Cu" "B.Cu") (free) (net 7))
+  (via (at 144.7 135) (size 0.6) (drill 0.3) (layers "F.Cu" "B.Cu") (free) (net 7))
+  (via (at 122.7 99.2) (size 0.6) (drill 0.3) (layers "F.Cu" "B.Cu") (free) (net 7))
   (via (at 131.4 112.5) (size 0.6) (drill 0.3) (layers "F.Cu" "B.Cu") (free) (net 7))
+  (via (at 151 96.8) (size 0.6) (drill 0.3) (layers "F.Cu" "B.Cu") (free) (net 7))
+  (via (at 120.4 104.7) (size 0.6) (drill 0.3) (layers "F.Cu" "B.Cu") (free) (net 7))
   (via (at 134.9 143.4) (size 0.6) (drill 0.3) (layers "F.Cu" "B.Cu") (free) (net 7))
+  (via (at 137.6 137) (size 0.6) (drill 0.3) (layers "F.Cu" "B.Cu") (free) (net 7))
+  (via (at 122.8 104.7) (size 0.6) (drill 0.3) (layers "F.Cu" "B.Cu") (free) (net 7))
+  (via (at 151 106.1) (size 0.6) (drill 0.3) (layers "F.Cu" "B.Cu") (free) (net 7))
   (via (at 116.4 134.4) (size 0.6) (drill 0.3) (layers "F.Cu" "B.Cu") (free) (net 7))
   (via (at 131.2 102.8) (size 0.6) (drill 0.3) (layers "F.Cu" "B.Cu") (free) (net 7))

Commit message: Schematic revision add decoupling cap on opamp
Changed lines of the file:
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@@
   (gr_line (start 115.8 91.6) (end 151.9 91.6) (layer "Edge.Cuts") (width 0.0381))
   (gr_line (start 115.76066 148.6) (end 152.3 148.6) (layer "Edge.Cuts") (width 0.0381))
-  (gr_arc (start 151.9 91.6) (mid 152.948087 91.98062) (end 153.4 93) (layer "Edge.Cuts") (width 0.0381))
+  (gr_arc (start 151.9 91.6) (mid 152.948088 91.98062) (end 153.4 93) (layer "Edge.Cuts") (width 0.0381))
   (gr_arc (start 153.4 147.4) (mid 153.131162 148.257732) (end 152.3 148.6) (layer "Edge.Cuts") (width 0.0381))
   (gr_line (start 114.3 93.4) (end 114.3 93.1) (layer "Edge.Cuts") (width 0.0381))

Commit message: v3 to production
Parts:
- removed J1: Conn_01x05_Male, Connector_PinSocket_2.54mm:PinSocket_1x05_P2.54mm_Vertical
- removed RV1, RV2, RV4: 10kA, Connector_PinHeader_2.54mm:PinHeader_1x03_P2.54mm_Vertical
- added Audio1: PJ-603A, AREA_lib_composant:AUDIO-TH_PJ-603A_1, B.Cu at (203.8, 72.8)
- added Audio2: PJ-603A, AREA_lib_composant:AUDIO-TH_PJ-603A_1, B.Cu at (199.2, 83.5)
- added C25: 100n, Capacitor_SMD:C_0603_1608Metric, F.Cu at (189.2, 105.0)
- added C26: 100n, Capacitor_SMD:C_0603_1608Metric, F.Cu at (189.2, 97.8)
- added C27: 100n, Capacitor_SMD:C_0603_1608Metric, F.Cu at (200.1, 94.3)
- added J2: Barrel_Jack_MountingPin, Connector_BarrelJack:BarrelJack_Horizontal, F.Cu at (201.8, 53.0)
- added R39: 0R, Resistor_SMD:R_0603_1608Metric, F.Cu at (206.8, 83.5)
- added R40: 0R, Resistor_SMD:R_0603_1608Metric, F.Cu at (196.2, 72.7)
- added R41: 10k, Resistor_SMD:R_0603_1608Metric, F.Cu at (192.2, 97.8)
- added R42: 10k, Resistor_SMD:R_0603_1608Metric, F.Cu at (195.2, 97.8)
- added SW1: ~, AREA_lib_composant:3PDT_LED, F.Cu at (201.5, 117.8)
- added kibuzzard-66C77FFB: G***, kibuzzard-66C77FFB, F.Cu at (216.4, 115.8)
- added kibuzzard-66C78013: G***, kibuzzard-66C78013, F.Cu at (210.1, 69.6)
- added kibuzzard-66C78027: G***, kibuzzard-66C78027, F.Cu at (193.5, 69.6)
- added kibuzzard-66C78076: G***, kibuzzard-66C78076, F.Cu at (210.1, 83.6)
- added kibuzzard-66C78083: G***, kibuzzard-66C78083, F.Cu at (192.9, 72.7)
- added kibuzzard-66C7864F: G***, kibuzzard-66C7864F, F.Cu at (201.2, 78.3)
- C1, C10, C11, C14, C15, C16, C17, C19, C20, C23, C3, C5, C6, C8, C9: footprint Capacitor_SMD:C_0805_2012Metric_Pad1.18x1.45mm_HandSolder -> Capacitor_SMD:C_0603_1608Metric
- C2, C21, C22, C24: footprint Capacitor_SMD:C_0805_2012Metric_Pad1.18x1.45mm_HandSolder -> Capacitor_SMD:C_0805_2012Metric
- D1: value BAT46 -> 1N5819WS; footprint Diode_SMD:D_SOD-123 -> Diode_SMD:D_SOD-323
- D2: value LED -> 1N5819WS; footprint LED_THT:LED_D3.0mm -> Diode_SMD:D_SOD-323
- D3, D4, D5, D8, D9: footprint Diode_SMD:D_SOD-123 -> Diode_SMD:D_SOD-323
- D6, D7: value BAT46 -> 1N4148; footprint Diode_SMD:D_SOD-123 -> Diode_SMD:D_SOD-323
- Q1: footprint Package_TO_SOT_SMD:SOT-323_SC-70_Handsoldering -> Package_TO_SOT_SMD:SOT-323_SC-70
- R1, R10, R11, R12, R13, R14, R15, R16, R17, R18, R19, R2, R20, R21, R22, R23, R24, R25, R26, R27, R28, R29, R3, R30, R31, R32, R33, R34, R35, R36, R37, R38, R4, R5, R6, R7, R9: footprint Resistor_SMD:R_0805_2012Metric_Pad1.20x1.40mm_HandSolder -> Resistor_SMD:R_0603_1608Metric
- R8: value 4k7 -> 1k; footprint Resistor_SMD:R_0805_2012Metric_Pad1.20x1.40mm_HandSolder -> Resistor_SMD:R_0603_1608Metric
- RV3: value 250kD -> 250k Log A; footprint Connector_PinHeader_2.54mm:PinHeader_1x03_P2.54mm_Vertical -> Potentiometer_THT:Potentiometer_Alpha_RD901F-40-00D_Single_Vertical
- RV5: footprint Connector_PinHeader_2.54mm:PinHeader_1x03_P2.54mm_Vertical -> Potentiometer_THT:Potentiometer_Alpha_RD901F-40-00D_Single_Vertical
- moved D2 128.3 mm to (208.5, 53.2), turned to 180 degrees
- moved D1 123.5 mm to (208.5, 51.2), turned to 180 degrees
- moved C4 123.2 mm to (211.5, 46.8)
- moved C7 114.6 mm to (191.5, 46.8), turned to 0 degrees
- moved R12 113.7 mm to (186.2, 48.8)
- moved R9 110.3 mm to (186.2, 50.2), turned to 180 degrees
- moved C12 102.4 mm to (215.5, 86.2), turned to 90 degrees
- moved RV3 96.1 mm to (205.9, 67.8), turned to 90 degrees
- moved R16 95.4 mm to (213.8, 95.7), turned to -90 degrees
- moved R18 95.0 mm to (213.0, 93.0)
- moved C9 94.9 mm to (212.2, 95.7), turned to 90 degrees
- moved Q1 92.4 mm to (217.0, 100.5)
- moved R15 92.1 mm to (217.0, 98.0)
- moved R8 91.8 mm to (210.2, 120.0), turned to 90 degrees
- moved Q2 91.6 mm to (216.5, 95.5)
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Connections:
- net /IN renamed /IN_FX
- net /OUT renamed /OUT_FX
- C10 pad 2: Net-(C10-Pad2) -> Net-(U2B--)
- C16 pad 2: Net-(C16-Pad2) -> Net-(U2B--)
- C2 pad 2: Net-(C2-Pad2) -> Net-(U2B--)
- C5 pad 2: Net-(C5-Pad2) -> Net-(U2B--)
- D2 pad 1: Net-(D2-Pad1) -> +9V
- D2 pad 2: +9V -> GND
- R25 pad 2: Net-(C16-Pad2) -> Net-(U2B--)
- R8 pad 1: /LED -> /IN_LED
- R8 pad 2: Net-(D2-Pad1) -> Net-(R8-Pad2)
- U2 pad 6: Net-(C16-Pad2) -> Net-(U2B--)
Routing:
- net Net-(C20-Pad2): track 16.4 -> 106.9 mm, vias 0 -> 1
- net Net-(C16-Pad2): track 77.8 -> 0.00 mm
- net +9V: track 113.0 -> 170.7 mm, vias 4 -> 9
- net /OUT: track 0.00 -> 56.0 mm
- net Net-(U2B-+): track 65.9 -> 18.5 mm
- net Net-(C13-Pad2): track 14.0 -> 53.2 mm, vias 0 -> 1
- net /IN: track 0.00 -> 32.9 mm
- net Net-(U2B--): track 0.00 -> 27.4 mm
- net Net-(R8-Pad2): track 0.00 -> 19.0 mm
- net Net-(C5-Pad2): track 16.4 -> 0.00 mm
- net Net-(C2-Pad2): track 15.0 -> 0.00 mm
- net Net-(C13-Pad1): track 18.6 -> 5.04 mm, vias 2 -> 0
- net Net-(U1B-+): track 22.6 -> 9.78 mm, vias 2 -> 0
- net /LED: track 12.5 -> 0.00 mm, vias 1 -> 0
- net Net-(Q3-C): track 22.9 -> 10.6 mm, vias 2 -> 0
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- added copper zone on F.Cu, net +9V
- added copper zone on F.Cu, net +BATT
- added copper zone on F.Cu, net /+4V5
- added copper zone on In1.Cu, net GND
- added copper zone on In2.Cu, net GND
Other:
- board size 39.1 x 57 mm -> 35 x 89.1 mm
- copper layers 2 -> 4
- board text added: "JLCJLCJLCJLC"
- board text removed: "9V"
- board text removed: "DIST"
- board text removed: "GND"
- board text removed: "HIGH"
- board text removed: "HM2 Clone V2"
- board text removed: "IN"
- board text removed: "LED"
- board text removed: "LOW"
- board text removed: "MID"
- board text removed: "OUT"
- board text removed: "VOL"

Commit message: V5 layout to review
Parts:
- removed D2: 1N5819WS, Diode_SMD:D_SOD-323
- removed Q4: 2SC2713, Package_TO_SOT_SMD:SOT-23
- removed R39, R40: 0R, Resistor_SMD:R_0603_1608Metric
- removed kibuzzard-66C77FFB: G***, kibuzzard-66C77FFB
- removed kibuzzard-66C78013: G***, kibuzzard-66C78013
- removed kibuzzard-66C78027: G***, kibuzzard-66C78027
- removed kibuzzard-66C78076: G***, kibuzzard-66C78076
- removed kibuzzard-66C78083: G***, kibuzzard-66C78083
- removed kibuzzard-66C7864F: G***, kibuzzard-66C7864F
- added C28: 100n, Capacitor_SMD:C_0603_1608Metric, F.Cu at (217.0, 51.0)
- added C29: 10n, Capacitor_SMD:C_0603_1608Metric, F.Cu at (217.0, 48.3)
- added Q5: 2N3904, Package_TO_SOT_SMD:SOT-23-3, F.Cu at (216.0, 109.5)
- Audio1, Audio2: moved to F.Cu
- C12: footprint Capacitor_SMD:CP_Elec_6.3x5.4 -> Capacitor_SMD:CP_Elec_4x5.8
- C4: value 100u -> 470u; footprint Capacitor_SMD:CP_Elec_6.3x7.7 -> Capacitor_SMD:CP_Elec_10x10
- C7: footprint Capacitor_SMD:CP_Elec_6.3x5.4 -> Capacitor_SMD:CP_Elec_6.3x5.8
- Q1: value 2SK880 -> MMBFJ201; footprint Package_TO_SOT_SMD:SOT-323_SC-70 -> Package_TO_SOT_SMD:SOT-23-3
- Q2: value 2SC2713 -> 2N3906; footprint Package_TO_SOT_SMD:SOT-23 -> Package_TO_SOT_SMD:SOT-23-3
- Q3: value 2SA1163 -> 2N3904; footprint Package_TO_SOT_SMD:SOT-23 -> Package_TO_SOT_SMD:SOT-23-3
- R32: value 470k -> 220k
- moved C18 43.6 mm to (202.0, 68.8)
- moved R31 34.7 mm to (197.5, 70.5)
- moved Q3 33.4 mm to (189.8, 118.2), turned to -90 degrees
- moved R22 31.9 mm to (212.5, 72.5)
- moved C15 29.6 mm to (209.5, 72.5), turned to 180 degrees
- moved C20 27.9 mm to (190.5, 114.7)
- moved C22 27.9 mm to (187.0, 118.2)
- moved R33 27.9 mm to (189.0, 114.7)
- moved R34 27.9 mm to (186.5, 113.9)
- moved R36 27.9 mm to (186.5, 115.4)
- moved R37 27.9 mm to (185.2, 118.2)
- moved C13 26.8 mm to (214.0, 76.2), turned to 0 degrees
- moved R20 26.5 mm to (215.5, 72.5), turned to 180 degrees
- moved TP1 24.0 mm to (190.8, 121.5)
- moved R14 20.5 mm to (210.0, 118.2), turned to 90 degrees
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Connections:
- Audio1 pad 4: Net-(Audio1-Pad4) -> /IN
- Audio1 pad 5: /OUT -> GND
- Audio2 pad 4: Net-(Audio2-Pad4) -> /OUT
- Audio2 pad 5: /IN -> GND
- C13 pad 1: Net-(C13-Pad1) -> Net-(Q5-C)
- C14 pad 1: Net-(Q2-C) -> Net-(Q5-C)
- C17 pad 1: Net-(Q3-C) -> Net-(Q2-C)
- C17 pad 2: Net-(Q3-B) -> Net-(Q2-B)
- C20 pad 1: Net-(Q4-B) -> Net-(Q3-B)
- C8 pad 1: Net-(Q1-S) -> Net-(Q1-D)
- C9 pad 1: Net-(Q2-B) -> Net-(Q5-B)
- C9 pad 2: Net-(Q2-C) -> Net-(Q5-C)
- Q1 pad 1: Net-(Q1-S) -> +9V
- Q1 pad 2: +9V -> Net-(Q1-D)
- Q2 pad 1: Net-(Q2-B) -> Net-(Q2-E)
- Q2 pad 2: Net-(Q2-E) -> Net-(Q2-B)
- Q3 pad 1: Net-(Q3-B) -> Net-(Q3-E)
- Q3 pad 2: Net-(Q3-E) -> Net-(Q3-B)
- Q3 pad 3: Net-(Q3-C) -> +9V
- R10 pad 1: Net-(Q1-S) -> Net-(Q1-D)
- R14 pad 2: Net-(Q2-B) -> Net-(Q5-B)
- R15 pad 2: Net-(Q2-B) -> Net-(Q5-B)
- R16 pad 1: Net-(Q2-C) -> Net-(Q5-C)
- R16 pad 2: Net-(Q2-B) -> Net-(Q5-B)
- R18 pad 2: Net-(Q2-C) -> Net-(Q5-C)
- R19 pad 2: Net-(Q2-E) -> Net-(Q5-E)
- R20 pad 1: Net-(C13-Pad1) -> Net-(R20-Pad1)
- R20 pad 2: Net-(Q2-C) -> Net-(C13-Pad2)
- R23 pad 2: Net-(Q3-B) -> Net-(Q2-B)
- R24 pad 2: Net-(Q3-B) -> Net-(Q2-B)
- R26 pad 1: Net-(Q3-C) -> Net-(Q2-C)
- R26 pad 2: Net-(Q3-B) -> Net-(Q2-B)
- R28 pad 1: Net-(Q3-E) -> Net-(Q2-E)
- R29 pad 2: Net-(Q3-C) -> Net-(Q2-C)
- R30 pad 1: Net-(Q3-C) -> Net-(Q2-C)
- R33 pad 2: Net-(Q4-B) -> Net-(Q3-B)
- R34 pad 1: Net-(Q4-E) -> Net-(Q3-E)
- R36 pad 1: Net-(Q4-E) -> Net-(Q3-E)
- R8 pad 1: /IN_LED -> +9V
- RV3 pad 1: Net-(C13-Pad2) -> Net-(R20-Pad1)
- SW1 pad 10: (no net) -> /GND_LED
- SW1 pad 12: GND -> (no net)
- SW1 pad 2: Net-(SW1-A-Pad1) -> /OUT
- SW1 pad 3: unconnected-(SW1-A-Pad3) -> /OUT_FX
- SW1 pad 4: /IN -> GND
- SW1 pad 5: /OUT -> GND
- SW1 pad 6: +9V -> /GND_LED
- SW1 pad 7: /IN_FX -> Net-(SW1-A-Pad1)
- SW1 pad 8: /OUT_FX -> /IN
- SW1 pad 9: /IN_LED -> /IN_FX
- U1 pad 3: Net-(Q3-C) -> Net-(Q2-C)
Routing:
- net Net-(C16-Pad1): track 8.98 -> 70.8 mm, vias 0 -> 2
- net Net-(C13-Pad2): track 53.2 -> 4.42 mm, vias 1 -> 0
- net Net-(Q5-C): track 0.00 -> 46.4 mm
- net Net-(C20-Pad2): track 106.9 -> 64.9 mm
- net Net-(R22-Pad2): track 39.8 -> 2.22 mm, vias 1 -> 0
- net Net-(R31-Pad1): track 46.3 -> 10.1 mm, vias 1 -> 0
- net /OUT: track 56.0 -> 24.0 mm
- net /GND_LED: track 0.00 -> 23.2 mm
- net Net-(C12-Pad1): track 13.8 -> 32.8 mm
- net Net-(U2B--): track 27.4 -> 45.0 mm, vias 0 -> 2
- net /+4V5: track 122.6 -> 139.9 mm, vias 7 -> 6
- net Net-(Q3-B): track 19.1 -> 3.20 mm
- net Net-(U2B-+): track 18.5 -> 33.5 mm
- net Net-(R20-Pad1): track 0.00 -> 14.4 mm
- net Net-(Q5-B): track 0.00 -> 12.8 mm
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Other:
- board size 35 x 89.1 mm -> 34 x 88.2 mm

Commit message: Added mecanical drawing and new pdf schem
v5 working
Parts:
- added C30: 100p, Capacitor_SMD:C_0603_1608Metric, F.Cu at (215.2, 84.7)
- added kibuzzard-66E86754: G***, kibuzzard-66E86754, F.Cu at (192.4, 67.8)
- added kibuzzard-66E8676F: G***, kibuzzard-66E8676F, F.Cu at (211.3, 68.2)
- added kibuzzard-66E8688E: G***, kibuzzard-66E8688E, F.Cu at (205.9, 83.8)
- C4: value 470u -> 220u; footprint Capacitor_SMD:CP_Elec_10x10 -> Capacitor_SMD:CP_Elec_6.3x7.7
- Q2: value 2N3906 -> MMBT3906; footprint Package_TO_SOT_SMD:SOT-23-3 -> Package_TO_SOT_SMD:SOT-23
- Q5: value 2N3904 -> MMBT3904; footprint Package_TO_SOT_SMD:SOT-23-3 -> Package_TO_SOT_SMD:SOT-23
- moved C29 2.83 mm to (217.1, 51.1), turned to 90 degrees
- moved C28 1.35 mm to (215.7, 51.1)
- moved C4 1.31 mm to (211.3, 51.3)
- moved Q2 0.65 mm to (211.4, 88.3), turned to -90 degrees
- moved Q5 0.31 mm to (215.7, 109.5), turned to 180 degrees
Connections:
- Q2 pad 1: Net-(Q2-E) -> Net-(Q2-B)
- Q2 pad 2: Net-(Q2-B) -> Net-(Q2-E)
- Q5 pad 1: Net-(Q5-E) -> Net-(Q5-B)
- Q5 pad 2: Net-(Q5-B) -> Net-(Q5-E)
- SW1 pad 12: (no net) -> /GND_LED
Routing:
- net /GND_LED: track 23.2 -> 30.2 mm
- net Net-(Q2-B): track 8.34 -> 14.5 mm
- net Net-(Q2-C): track 25.1 -> 30.1 mm
- net Net-(Q5-C): track 46.4 -> 44.3 mm
- net Net-(C5-Pad1): track 20.4 -> 22.4 mm
- net Net-(Q2-E): track 4.65 -> 2.74 mm
- net Net-(Q5-B): track 12.8 -> 14.4 mm
- net Net-(Q5-E): track 1.58 -> 3.18 mm
- net Net-(C20-Pad2): track 64.9 -> 66.3 mm
- net GND: track 0.00 -> 1.16 mm, vias 170 -> 173
- net +9V: track 176.5 -> 177.3 mm
- net Net-(C16-Pad1): track 70.8 -> 71.4 mm
- removed copper zone on In1.Cu, net GND
- removed copper zone on In2.Cu, net GND
Other:
- board size 34 x 88.2 mm -> 34 x 88 mm
- copper layers 4 -> 2
